File: cd4046be_new_educational_pcb/rf.kicad_sch (KiCad schematic)
At the start: 9 parts, among them IC1 CD4046BE, J1 Conn_01x02_Socket, J2 Conn_01x08_Socket, J3 Conn_01x08_Socket, J4 Conn_01x02_Socket, J5 Conn_01x02_Socket, J6 Conn_01x02_Socket, J7 Conn_01x02_Socket, J8 Conn_01x02_Socket

Commit message: a
Parts:
- IC1: footprint KiCad:DIP794W53P254L1930H508Q16N -> Package_DIP:CERDIP-16_W7.62mm_SideBrazed
Changed lines of the file:
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@@
 			)
 		)
-		(property "Footprint" "KiCad:DIP794W53P254L1930H508Q16N"
+		(property "Footprint" "Package_DIP:CERDIP-16_W7.62mm_SideBrazed"
 			(at 165.1 144.45 0)
 			(effects

Commit message: α
Parts:
- added J9: Conn_01x02_Socket, Connector_PinSocket_2.54mm:PinSocket_1x02_P2.54mm_Vertical, symbol Connector:Conn_01x02_Socket
Connections:
- net GND: now also J9.1 (Pin_1), J9.2 (Pin_2)
Changed lines of the file:
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@@
 	(wire
 		(pts
-			(xy 104.14 34.29) (xy 116.84 34.29)
+			(xy 96.52 26.67) (xy 109.22 26.67)
 		)
 		(stroke
@@
 	)
 	(label "GND"
+		(at 195.58 59.69 0)
+		(effects
+			(font
+				(size 1.27 1.27)
+			)
+			(justify left bottom)
+		)
+	)
+	(label "GND"
 		(at 101.6 67.31 0)
 		(effects
@@
 	(label "PC1"
 		(at 100.33 52.07 0)
+		(effects
+			(font
+				(size 1.27 1.27)
+			)
+			(justify left bottom)
+		)
+	)
+	(label "GND"
+		(at 195.58 62.23 0)
 		(effects
 			(font
@@
 	(symbol
 		(lib_id "power:VDD")
-		(at 104.14 34.29 0)
+		(at 96.52 26.67 0)
 		(unit 1)
 		(exclude_from_sim no)
@@
 		(fields_autoplaced yes)
 		(property "Reference" "#PWR02"
-			(at 104.14 38.1 0)
+			(at 96.52 30.48 0)
 			(effects
 				(font
@@
 		)
 		(property "Value" "VDD"
-			(at 104.14 29.21 0)
+			(at 96.52 21.59 0)
 			(effects
 				(font
@@
 		)
 		(property "Footprint" ""
-			(at 104.14 34.29 0)
+			(at 96.52 26.67 0)
 			(effects
 				(font
@@
 		)
 		(property "Datasheet" ""
-			(at 104.14 34.29 0)
+			(at 96.52 26.67 0)
 			(effects
 				(font
@@
 		)
 		(property "Description" "Power symbol creates a global label with name \"VDD\""
-			(at 104.14 34.29 0)
+			(at 96.52 26.67 0)
 			(effects
 				(font
@@
 	(symbol
 		(lib_id "power:GND")
-		(at 91.44 34.29 0)
+		(at 78.74 29.21 0)
 		(unit 1)
 		(exclude_from_sim no)
@@
 		(fields_autoplaced yes)
 		(property "Reference" "#PWR01"
-			(at 91.44 40.64 0)
+			(at 78.74 35.56 0)
 			(effects
 				(font
@@
 		)
 		(property "Value" "GND"
-			(at 91.44 39.37 0)
+			(at 78.74 34.29 0)
 			(effects
 				(font
@@
 		)
 		(property "Footprint" ""
-			(at 91.44 34.29 0)
+			(at 78.74 29.21 0)
 			(effects
 				(font
@@
 		)
 		(property "Datasheet" ""
-			(at 91.44 34.29 0)
+			(at 78.74 29.21 0)
 			(effects
 				(font
@@
 		)
 		(property "Description" "Power symbol creates a global label with name \"GND\" , ground"
-			(at 91.44 34.29 0)
+			(at 78.74 29.21 0)
 			(effects
 				(font
@@
 	(symbol
 		(lib_id "Connector:Conn_01x02_Socket")
+		(at 200.66 59.69 0)
+		(unit 1)
+		(exclude_from_sim no)
+		(in_bom yes)
+		(on_board yes)
+		(dnp no)
+		(fields_autoplaced yes)
+		(property "Reference" "J9"
+			(at 201.93 59.6899 0)
+			(effects
+				(font
+					(size 1.27 1.27)
+				)
+				(justify left)
+			)
+		)
+		(property "Value" "Conn_01x02_Socket"
+			(at 201.93 62.2299 0)
+			(effects
+				(font
+					(size 1.27 1.27)
+				)
+				(justify left)
+			)
+		)
+		(property "Footprint" "Connector_PinSocket_2.54mm:PinSocket_1x02_P2.54mm_Vertical"
+			(at 200.66 59.69 0)
+			(effects
+				(font
+					(size 1.27 1.27)
+				)
+				(hide yes)
+			)
+		)
+		(property "Datasheet" "~"
+			(at 200.66 59.69 0)
+			(effects
+				(font
+					(size 1.27 1.27)
+				)
+				(hide yes)
+			)
+		)
+		(property "Description" "Generic connector, single row, 01x02, script generated"
+			(at 200.66 59.69 0)
+			(effects
+				(font
+					(size 1.27 1.27)
+				)
+				(hide yes)
+			)
+		)
+		(pin "2"
+		)
+		(pin "1"
+		)
+		(instances
+			(project ""
+				(path "/bd49dab0-12b6-4327-a1c4-25d038404486"
+					(reference "J9")
+					(unit 1)
+				)
+			)
+		)
+	)
+	(symbol
+		(lib_id "Connector:Conn_01x02_Socket")
 		(at 128.27 96.52 0)
 		(unit 1)
@@
 	(symbol
 		(lib_id "power:PWR_FLAG")
-		(at 116.84 34.29 0)
+		(at 109.22 26.67 0)
 		(unit 1)
 		(exclude_from_sim no)
@@
 		(fields_autoplaced yes)
 		(property "Reference" "#FLG02"
-			(at 116.84 32.385 0)
+			(at 109.22 24.765 0)
 			(effects
 				(font
@@
 		)
 		(property "Value" "PWR_FLAG"
-			(at 116.84 29.21 0)
+			(at 109.22 21.59 0)
 			(effects
 				(font
@@
 		)
 		(property "Footprint" ""
-			(at 116.84 34.29 0)
+			(at 109.22 26.67 0)
 			(effects
 				(font
@@
 		)
 		(property "Datasheet" "~"
-			(at 116.84 34.29 0)
+			(at 109.22 26.67 0)
 			(effects
 				(font
@@
 		)
 		(property "Description" "Special symbol for telling ERC where power comes from"
-			(at 116.84 34.29 0)
+			(at 109.22 26.67 0)
 			(effects
 				(font
@@
 	(symbol
 		(lib_id "power:PWR_FLAG")
-		(at 91.44 34.29 0)
+		(at 78.74 29.21 0)
 		(unit 1)
 		(exclude_from_sim no)
@@
 		(fields_autoplaced yes)
 		(property "Reference" "#FLG01"
-			(at 91.44 32.385 0)
+			(at 78.74 27.305 0)
 			(effects
 				(font
@@
 		)
 		(property "Value" "PWR_FLAG"
-			(at 91.44 29.21 0)
+			(at 78.74 24.13 0)
 			(effects
 				(font
@@
 		)
 		(property "Footprint" ""
-			(at 91.44 34.29 0)
+			(at 78.74 29.21 0)
 			(effects
 				(font
@@
 		)
 		(property "Datasheet" "~"
-			(at 91.44 34.29 0)
+			(at 78.74 29.21 0)
 			(effects
 				(font
@@
 		)
 		(property "Description" "Special symbol for telling ERC where power comes from"
-			(at 91.44 34.29 0)
-			(effects
-				(font
+			(at 78.74 29.21 0)
+			(effects
+				(font
