File: cd4046be_new_educational_pcb/rf.kicad_pcb (KiCad board)
At the start: 2 copper layers, 27.5 x 39.5 mm, 9 parts, among them IC1 CD4046BE, J1 Conn_01x02_Socket, J2 Conn_01x08_Socket, J3 Conn_01x08_Socket, J4 Conn_01x02_Socket, J5 Conn_01x02_Socket, J6 Conn_01x02_Socket, J7 Conn_01x02_Socket, J8 Conn_01x02_Socket

Commit message: a
Parts:
- added IC1: CD4046BE, KiCad:DIP794W53P254L1930H508Q16N, F.Cu at (154.0, 127.0)
- added IC1: CD4046BE, KiCad:DIP794W53P254L1930H508Q16N, F.Cu at (197.8, 94.5)
- added IC1: CD4046BE, KiCad:DIP794W53P254L1930H508Q16N, F.Cu at (197.2, 126.8)
- added J1: Conn_01x02_Socket, Connector_PinSocket_2.54mm:PinSocket_1x02_P2.54mm_Vertical, F.Cu at (137.6, 118.2)
- added J1: Conn_01x02_Socket, Connector_PinSocket_2.54mm:PinSocket_1x02_P2.54mm_Vertical, F.Cu at (180.9, 118.0)
- added J1: Conn_01x02_Socket, Connector_PinSocket_2.54mm:PinSocket_1x02_P2.54mm_Vertical, F.Cu at (181.4, 85.7)
- added J2: Conn_01x08_Socket, Connector_PinSocket_2.54mm:PinSocket_1x08_P2.54mm_Vertical, F.Cu at (162.8, 118.2)
- added J2: Conn_01x08_Socket, Connector_PinSocket_2.54mm:PinSocket_1x08_P2.54mm_Vertical, F.Cu at (206.0, 118.0)
- added J2: Conn_01x08_Socket, Connector_PinSocket_2.54mm:PinSocket_1x08_P2.54mm_Vertical, F.Cu at (206.5, 85.8)
- added J3: Conn_01x08_Socket, Connector_PinSocket_2.54mm:PinSocket_1x08_P2.54mm_Vertical, F.Cu at (162.8, 135.5)
- added J3: Conn_01x08_Socket, Connector_PinSocket_2.54mm:PinSocket_1x08_P2.54mm_Vertical, F.Cu at (206.0, 135.2)
- added J3: Conn_01x08_Socket, Connector_PinSocket_2.54mm:PinSocket_1x08_P2.54mm_Vertical, F.Cu at (206.5, 103.0)
- added J4: Conn_01x02_Socket, Connector_PinSocket_2.54mm:PinSocket_1x02_P2.54mm_Vertical, F.Cu at (181.1, 123.7)
- added J4: Conn_01x02_Socket, Connector_PinSocket_2.54mm:PinSocket_1x02_P2.54mm_Vertical, F.Cu at (137.9, 124.0)
- added J4: Conn_01x02_Socket, Connector_PinSocket_2.54mm:PinSocket_1x02_P2.54mm_Vertical, F.Cu at (181.6, 91.5)
- added J5: Conn_01x02_Socket, Connector_PinSocket_2.54mm:PinSocket_1x02_P2.54mm_Vertical, F.Cu at (130.1, 124.0)
- added J5: Conn_01x02_Socket, Connector_PinSocket_2.54mm:PinSocket_1x02_P2.54mm_Vertical, F.Cu at (173.4, 123.7)
- added J5: Conn_01x02_Socket, Connector_PinSocket_2.54mm:PinSocket_1x02_P2.54mm_Vertical, F.Cu at (173.9, 91.5)
- added J6: Conn_01x02_Socket, Connector_PinSocket_2.54mm:PinSocket_1x02_P2.54mm_Vertical, F.Cu at (182.1, 101.7)
- added J6: Conn_01x02_Socket, Connector_PinSocket_2.54mm:PinSocket_1x02_P2.54mm_Vertical, F.Cu at (181.6, 134.0)
- added J6: Conn_01x02_Socket, Connector_PinSocket_2.54mm:PinSocket_1x02_P2.54mm_Vertical, F.Cu at (138.4, 134.2)
- added J7: Conn_01x02_Socket, Connector_PinSocket_2.54mm:PinSocket_1x02_P2.54mm_Vertical, F.Cu at (130.6, 138.7)
- added J7: Conn_01x02_Socket, Connector_PinSocket_2.54mm:PinSocket_1x02_P2.54mm_Vertical, F.Cu at (173.9, 138.5)
- added J7: Conn_01x02_Socket, Connector_PinSocket_2.54mm:PinSocket_1x02_P2.54mm_Vertical, F.Cu at (174.4, 106.2)
- added J8: Conn_01x02_Socket, Connector_PinSocket_2.54mm:PinSocket_1x02_P2.54mm_Vertical, F.Cu at (138.4, 138.7)
- added J8: Conn_01x02_Socket, Connector_PinSocket_2.54mm:PinSocket_1x02_P2.54mm_Vertical, F.Cu at (182.1, 106.2)
- added J8: Conn_01x02_Socket, Connector_PinSocket_2.54mm:PinSocket_1x02_P2.54mm_Vertical, F.Cu at (181.6, 138.5)
- moved J2 28.0 mm to (162.9, 86.3), turned to -90 degrees
- moved J3 27.5 mm to (162.9, 103.5), turned to -90 degrees
- moved J7 26.2 mm to (130.8, 106.8), turned to -90 degrees
- moved J5 21.7 mm to (130.2, 92.0), turned to -90 degrees
- moved J8 18.9 mm to (138.5, 106.8), turned to -90 degrees
- moved J1 16.6 mm to (137.8, 86.2), turned to 180 degrees
- moved J6 13.8 mm to (138.5, 102.2), turned to 180 degrees
- moved IC1 12.6 mm to (154.1, 95.1), turned to -90 degrees
- moved J4 11.2 mm to (138.0, 92.0), turned to -90 degrees
Routing:
- net /VCO_IN: track 41.7 -> 166.6 mm
- net GND: track 40.6 -> 162.4 mm
- net /PC1: track 28.5 -> 114.1 mm
- net /PC2: track 25.6 -> 102.5 mm
- net Net-(J7-Pin_1): track 5.21 -> 20.8 mm
- net Net-(J4-Pin_2): track 5.21 -> 20.8 mm
- net Net-(IC1-COMPARATOR_IN): track 4.87 -> 19.5 mm
- net Net-(IC1-CI(2)): track 4.87 -> 19.5 mm
- net Net-(IC1-VCO_OUT): track 4.87 -> 19.5 mm
- net Net-(IC1-CI(1)): track 4.87 -> 19.5 mm
- net Net-(IC1-PHASE_PULSES): track 4.87 -> 19.5 mm
- net Net-(IC1-INHIBIT): track 4.87 -> 19.5 mm
- net Net-(IC1-DEMODULATOR_OUT): track 4.56 -> 18.2 mm
- net Net-(IC1-SIGNAL_IN): track 4.56 -> 18.2 mm
- net Net-(IC1-R2_TO_VSS): track 4.56 -> 18.2 mm
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Other:
- board size 27.5 x 39.5 mm -> 84.5 x 60.5 mm

Commit message: α
Parts:
- removed the IC1 at (154.0, 127.0)
- removed the IC1 at (197.8, 94.5)
- removed the IC1 at (197.2, 126.8)
- removed the IC1 at (154.1, 95.1)
- removed the J1 at (137.6, 118.2)
- removed the J1 at (180.9, 118.0)
- removed the J1 at (181.4, 85.7)
- removed the J1 at (137.8, 86.2)
- removed the J2 at (162.8, 118.2)
- removed the J2 at (162.9, 86.3)
- removed the J2 at (206.0, 118.0)
- removed the J2 at (206.5, 85.8)
- removed the J3 at (162.8, 135.5)
- removed the J3 at (206.0, 135.2)
- removed the J3 at (162.9, 103.5)
- removed the J3 at (206.5, 103.0)
- removed the J4 at (181.1, 123.7)
- removed the J4 at (137.9, 124.0)
- removed the J4 at (181.6, 91.5)
- removed the J4 at (138.0, 92.0)
- removed the J5 at (130.2, 92.0)
- removed the J5 at (130.1, 124.0)
- removed the J5 at (173.4, 123.7)
- removed the J5 at (173.9, 91.5)
- removed the J6 at (182.1, 101.7)
- removed the J6 at (181.6, 134.0)
- removed the J6 at (138.4, 134.2)
- removed the J6 at (138.5, 102.2)
- removed the J7 at (130.6, 138.7)
- removed the J7 at (130.8, 106.8)
- removed the J7 at (173.9, 138.5)
- removed the J7 at (174.4, 106.2)
- removed the J8 at (138.4, 138.7)
- removed the J8 at (182.1, 106.2)
- removed the J8 at (181.6, 138.5)
- removed the J8 at (138.5, 106.8)
- added IC1: CD4046BE, Package_DIP:CERDIP-16_W7.62mm_SideBrazed, F.Cu at (171.9, 87.4)
- added J1: Conn_01x02_Socket, Connector_PinSocket_2.54mm:PinSocket_1x02_P2.54mm_Vertical, F.Cu at (146.8, 82.5)
- added J2: Conn_01x08_Socket, Connector_PinSocket_2.54mm:PinSocket_1x08_P2.54mm_Vertical, F.Cu at (171.9, 82.5)
- added J3: Conn_01x08_Socket, Connector_PinSocket_2.54mm:PinSocket_1x08_P2.54mm_Vertical, F.Cu at (171.9, 99.8)
- added J4: Conn_01x02_Socket, Connector_PinSocket_2.54mm:PinSocket_1x02_P2.54mm_Vertical, F.Cu at (147.0, 88.2)
- added J5: Conn_01x02_Socket, Connector_PinSocket_2.54mm:PinSocket_1x02_P2.54mm_Vertical, F.Cu at (139.2, 88.2)
- added J6: Conn_01x02_Socket, Connector_PinSocket_2.54mm:PinSocket_1x02_P2.54mm_Vertical, F.Cu at (147.5, 98.5)
- added J7: Conn_01x02_Socket, Connector_PinSocket_2.54mm:PinSocket_1x02_P2.54mm_Vertical, F.Cu at (140.0, 101.8)
- added J8: Conn_01x02_Socket, Connector_PinSocket_2.54mm:PinSocket_1x02_P2.54mm_Vertical, F.Cu at (148.2, 102.5)
- added J9: Conn_01x02_Socket, Connector_PinSocket_2.54mm:PinSocket_1x02_P2.54mm_Vertical, F.Cu at (159.2, 103.5)
Routing:
- net /VCO_IN: track 166.6 -> 40.7 mm
- net /PC1: track 114.1 -> 28.5 mm
- net /PC2: track 102.5 -> 25.6 mm
- net GND: track 162.4 -> 98.4 mm
- net Net-(J4-Pin_2): track 20.8 -> 5.21 mm
- net Net-(J7-Pin_1): track 20.8 -> 6.01 mm
- net Net-(IC1-VCO_OUT): track 19.5 -> 4.87 mm
- net Net-(IC1-COMPARATOR_IN): track 19.5 -> 4.87 mm
- net Net-(IC1-CI(2)): track 19.5 -> 4.87 mm
- net Net-(IC1-PHASE_PULSES): track 19.5 -> 4.87 mm
- net Net-(IC1-INHIBIT): track 19.5 -> 4.87 mm
- net Net-(IC1-CI(1)): track 19.5 -> 4.87 mm
- net Net-(IC1-SIGNAL_IN): track 18.2 -> 4.56 mm
- net Net-(IC1-DEMODULATOR_OUT): track 18.2 -> 4.56 mm
- net VDD: track 18.2 -> 4.56 mm
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Other:
- board size 84.5 x 60.5 mm -> 44.5 x 32 mm

Commit message: α
Parts:
- removed the IC1 at (171.9, 87.4)
- removed the J1 at (146.8, 82.5)
- removed the J2 at (171.9, 82.5)
- removed the J3 at (171.9, 99.8)
- removed the J4 at (147.0, 88.2)
- removed the J5 at (139.2, 88.2)
- removed the J6 at (147.5, 98.5)
- removed the J7 at (140.0, 101.8)
- removed the J8 at (148.2, 102.5)
- removed the J9 at (159.2, 103.5)
- added IC1: CD4046BE, Package_DIP:CERDIP-16_W7.62mm_SideBrazed, F.Cu at (171.9, 51.9)
- added IC1: CD4046BE, Package_DIP:CERDIP-16_W7.62mm_SideBrazed, F.Cu at (221.4, 51.9)
- added J1: Conn_01x02_Socket, Connector_PinSocket_2.54mm:PinSocket_1x02_P2.54mm_Vertical, F.Cu at (196.2, 47.0)
- added J1: Conn_01x02_Socket, Connector_PinSocket_2.54mm:PinSocket_1x02_P2.54mm_Vertical, F.Cu at (146.8, 47.0)
- added J2: Conn_01x08_Socket, Connector_PinSocket_2.54mm:PinSocket_1x08_P2.54mm_Vertical, F.Cu at (171.9, 47.0)
- added J2: Conn_01x08_Socket, Connector_PinSocket_2.54mm:PinSocket_1x08_P2.54mm_Vertical, F.Cu at (221.4, 47.0)
- added J3: Conn_01x08_Socket, Connector_PinSocket_2.54mm:PinSocket_1x08_P2.54mm_Vertical, F.Cu at (221.4, 64.3)
- added J3: Conn_01x08_Socket, Connector_PinSocket_2.54mm:PinSocket_1x08_P2.54mm_Vertical, F.Cu at (171.9, 64.3)
- added J4: Conn_01x02_Socket, Connector_PinSocket_2.54mm:PinSocket_1x02_P2.54mm_Vertical, F.Cu at (147.0, 52.8)
- added J4: Conn_01x02_Socket, Connector_PinSocket_2.54mm:PinSocket_1x02_P2.54mm_Vertical, F.Cu at (196.5, 52.8)
- added J5: Conn_01x02_Socket, Connector_PinSocket_2.54mm:PinSocket_1x02_P2.54mm_Vertical, F.Cu at (139.2, 52.8)
- added J5: Conn_01x02_Socket, Connector_PinSocket_2.54mm:PinSocket_1x02_P2.54mm_Vertical, F.Cu at (188.8, 52.8)
- added J6: Conn_01x02_Socket, Connector_PinSocket_2.54mm:PinSocket_1x02_P2.54mm_Vertical, F.Cu at (147.5, 63.0)
- added J6: Conn_01x02_Socket, Connector_PinSocket_2.54mm:PinSocket_1x02_P2.54mm_Vertical, F.Cu at (197.0, 63.0)
- added J7: Conn_01x02_Socket, Connector_PinSocket_2.54mm:PinSocket_1x02_P2.54mm_Vertical, F.Cu at (189.5, 66.3)
- added J7: Conn_01x02_Socket, Connector_PinSocket_2.54mm:PinSocket_1x02_P2.54mm_Vertical, F.Cu at (140.0, 66.3)
- added J8: Conn_01x02_Socket, Connector_PinSocket_2.54mm:PinSocket_1x02_P2.54mm_Vertical, F.Cu at (197.8, 67.0)
- added J8: Conn_01x02_Socket, Connector_PinSocket_2.54mm:PinSocket_1x02_P2.54mm_Vertical, F.Cu at (148.2, 67.0)
- added J9: Conn_01x02_Socket, Connector_PinSocket_2.54mm:PinSocket_1x02_P2.54mm_Vertical, F.Cu at (159.2, 68.0)
- added J9: Conn_01x02_Socket, Connector_PinSocket_2.54mm:PinSocket_1x02_P2.54mm_Vertical, F.Cu at (208.8, 68.0)
Routing:
- net GND: track 98.4 -> 196.8 mm
- net /VCO_IN: track 40.7 -> 73.9 mm
- net /PC1: track 28.5 -> 57.0 mm
- net /PC2: track 25.6 -> 51.2 mm
- net Net-(J7-Pin_1): track 6.01 -> 12.0 mm
- net Net-(J4-Pin_2): track 5.21 -> 10.4 mm
- net Net-(IC1-VCO_OUT): track 4.87 -> 9.74 mm
- net Net-(IC1-COMPARATOR_IN): track 4.87 -> 9.74 mm
- net Net-(IC1-CI(2)): track 4.87 -> 9.74 mm
- net Net-(IC1-PHASE_PULSES): track 4.87 -> 9.74 mm
- net Net-(IC1-INHIBIT): track 4.87 -> 9.74 mm
- net Net-(IC1-CI(1)): track 4.87 -> 9.74 mm
- net Net-(IC1-SIGNAL_IN): track 4.56 -> 9.12 mm
- net Net-(IC1-DEMODULATOR_OUT): track 4.56 -> 9.12 mm
- net VDD: track 4.56 -> 9.12 mm
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Other:
- board size 44.5 x 32 mm -> 94 x 32 mm
