File: cd4046be_new_educational_pcb/rf.kicad_pcb (KiCad board)
At the start: 2 copper layers, 94 x 32 mm, 20 parts, among them IC1 CD4046BE, J1 Conn_01x02_Socket, J2 Conn_01x08_Socket, J3 Conn_01x08_Socket, J4 Conn_01x02_Socket, J5 Conn_01x02_Socket, J6 Conn_01x02_Socket, J7 Conn_01x02_Socket, J8 Conn_01x02_Socket, J9 Conn_01x02_Socket

Commit message: ?
Parts:
- removed the IC1 at (221.4, 51.9)
- removed the J1 at (196.2, 47.0)
- removed the J2 at (221.4, 47.0)
- removed the J3 at (221.4, 64.3)
- removed the J4 at (196.5, 52.8)
- removed the J5 at (188.8, 52.8)
- removed the J6 at (197.0, 63.0)
- removed the J7 at (189.5, 66.3)
- removed the J8 at (197.8, 67.0)
- removed the J9 at (208.8, 68.0)
Routing:
- net GND: track 196.8 -> 98.4 mm
- net /VCO_IN: track 73.9 -> 36.9 mm
- net /PC1: track 57.0 -> 28.5 mm
- net /PC2: track 51.2 -> 25.6 mm
- net Net-(J7-Pin_1): track 12.0 -> 6.01 mm
- net Net-(J4-Pin_2): track 10.4 -> 5.21 mm
- net Net-(IC1-VCO_OUT): track 9.74 -> 4.87 mm
- net Net-(IC1-COMPARATOR_IN): track 9.74 -> 4.87 mm
- net Net-(IC1-CI(2)): track 9.74 -> 4.87 mm
- net Net-(IC1-PHASE_PULSES): track 9.74 -> 4.87 mm
- net Net-(IC1-INHIBIT): track 9.74 -> 4.87 mm
- net Net-(IC1-CI(1)): track 9.74 -> 4.87 mm
- net Net-(IC1-SIGNAL_IN): track 9.12 -> 4.56 mm
- net Net-(IC1-DEMODULATOR_OUT): track 9.12 -> 4.56 mm
- net VDD: track 9.12 -> 4.56 mm
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Other:
- board size 94 x 32 mm -> 44.5 x 32 mm

Commit message: a
Routing:
- net /PC1: track 28.5 -> 29.7 mm
- net /PC2: track 25.6 -> 26.7 mm
