File: cd4046be_new_educational_pcb/teliko.kicad_sch (KiCad schematic)
At the start: 10 parts, among them IC1 CD4046BE, J1 Conn_01x02_Socket, J2 Conn_01x08_Socket, J3 Conn_01x08_Socket, J4 Conn_01x02_Socket, J5 Conn_01x02_Socket, J6 Conn_01x02_Socket, J7 Conn_01x02_Socket, J8 Conn_01x02_Socket, J9 Conn_01x02_Socket

Commit message: l
Parts:
- added J10: Conn_01x01_Socket, Connector_PinSocket_2.54mm:PinSocket_1x01_P2.54mm_Vertical, symbol Connector:Conn_01x01_Socket
Connections:
- net GND: now also J10.1 (Pin_1)
